Commit message: chore(ci): added rrbot dataset for ci pipeline

File: atom_examples/rrbot/rrbot_calibration/urdf/optimized.urdf.xacro (robot description, xacro)
@@ -12,5 +12,5 @@
   </gazebo>
   <joint name="rgb_left_joint" type="fixed">
-    <origin xyz="0.01499999999999957 -3.2057426077360894e-16 0.012000000000000375" rpy="-3.0805097672264623e-16 4.385950745910349e-16 2.603825111285602e-17"/>
+    <origin xyz="0.015423429555058824 -0.004097649647616211 0.015355858307271672" rpy="-0.0022587392426797995 0.0022602207514791357 0.002967983406372327"/>
     <parent link="tripod_left_support"/>
     <child link="rgb_left_link"/>
@@ -80,5 +80,5 @@
   </gazebo>
   <joint name="rgb_right_joint" type="fixed">
-    <origin xyz="0.014896101514833615 -0.00010643945277278731 0.011919487541689396" rpy="-9.733722284792457e-05 -8.500523015444027e-05 7.164825060903521e-05"/>
+    <origin xyz="0.01289213581339572 0.003326035608129313 0.008356055368279793" rpy="-0.0006387747062078774 -0.003016395599784455 -0.0027341872079828296"/>
     <parent link="tripod_right_support"/>
     <child link="rgb_right_link"/>
