Commit message: fix(ci): fixed riwbot dataset with correct pattern name

File: atom_examples/riwbot/riwbot_calibration/urdf/optimized.urdf.xacro (robot description, xacro)
@@ -555,5 +555,5 @@
   </joint>
   <joint name="rgb_world_joint" type="fixed">
-    <origin xyz="0.00018422549328598914 -8.687126147423204e-05 0.03082428267298673" rpy="1.782480977365134e-05 0.0008392950298426041 -6.424682384297097e-05"/>
+    <origin xyz="0.00016217990171165565 -7.145197012276274e-05 0.029180073996584944" rpy="0.00010608885856825412 -0.0005218577838252585 -0.00027747251278555817"/>
     <parent link="tripod_center_support"/>
     <child link="rgb_world_link"/>

File: atom_examples/riwbot/riwbot_calibration/urdf/optimized_w_pattern.urdf.xacro (robot description, xacro)
@@ -555,5 +555,5 @@
   </joint>
   <joint name="rgb_world_joint" type="fixed">
-    <origin xyz="0.00018422549328598914 -8.687126147423204e-05 0.03082428267298673" rpy="1.782480977365134e-05 0.0008392950298426041 -6.424682384297097e-05"/>
+    <origin xyz="0.00016217990171165565 -7.145197012276274e-05 0.029180073996584944" rpy="0.00010608885856825412 -0.0005218577838252585 -0.00027747251278555817"/>
     <parent link="tripod_center_support"/>
     <child link="rgb_world_link"/>
@@ -646,5 +646,5 @@
     <child link="charuco_200x200_4x4"/>
   </joint>
-  <link name="pattern_link">
+  <link name="charuco_200x200_4x4">
     <origin xyz="0 0 0" rpy="0 0 0"/>
     <visual name="pattern_1_visual">
@@ -655,8 +655,8 @@
     </visual>
   </link>
-  <joint name="flange-pattern_link" type="fixed">
-    <origin xyz="0.05983295925390568 -0.06028112203976766 0.0006639433404215635" rpy="-0.0008146576348299466 -6.542257039450517e-05 -0.00021449988423033597"/>
+  <joint name="flange-charuco_200x200_4x4" type="fixed">
+    <origin xyz="0.06017527282800442 -0.05972593502907463 0.0005492165842738227" rpy="0.0001526206514825427 -0.0012433053112463365 0.0006108917325790478"/>
     <parent link="flange"/>
-    <child link="pattern_link"/>
+    <child link="charuco_200x200_4x4"/>
   </joint>
 </robot>

Commit message: chore(ci): cleared up main pipeline

File: atom_examples/riwbot/riwbot_calibration/urdf/optimized.urdf.xacro (robot description, xacro)
@@ -555,5 +555,5 @@
   </joint>
   <joint name="rgb_world_joint" type="fixed">
-    <origin xyz="0.00016217990171165565 -7.145197012276274e-05 0.029180073996584944" rpy="0.00010608885856825412 -0.0005218577838252585 -0.00027747251278555817"/>
+    <origin xyz="3.906898692642251e-05 -0.0001141153593696933 0.0296251830600485" rpy="3.641044641491813e-05 4.391475742434813e-05 -0.0001714502119169957"/>
     <parent link="tripod_center_support"/>
     <child link="rgb_world_link"/>

File: atom_examples/riwbot/riwbot_calibration/urdf/optimized_w_pattern.urdf.xacro (robot description, xacro)
@@ -555,5 +555,5 @@
   </joint>
   <joint name="rgb_world_joint" type="fixed">
-    <origin xyz="0.00016217990171165565 -7.145197012276274e-05 0.029180073996584944" rpy="0.00010608885856825412 -0.0005218577838252585 -0.00027747251278555817"/>
+    <origin xyz="3.906898692642251e-05 -0.0001141153593696933 0.0296251830600485" rpy="3.641044641491813e-05 4.391475742434813e-05 -0.0001714502119169957"/>
     <parent link="tripod_center_support"/>
     <child link="rgb_world_link"/>
@@ -656,5 +656,5 @@
   </link>
   <joint name="flange-charuco_200x200_4x4" type="fixed">
-    <origin xyz="0.06017527282800442 -0.05972593502907463 0.0005492165842738227" rpy="0.0001526206514825427 -0.0012433053112463365 0.0006108917325790478"/>
+    <origin xyz="0.06015956044003661 -0.05967715702177562 0.00048249876383632626" rpy="0.0001426487145295442 -0.0009698348622317083 0.0004909416845332869"/>
     <parent link="flange"/>
     <child link="charuco_200x200_4x4"/>
